File: cornMerge/cornMerge.brd (EAGLE design)
At the start: 101.6 x 49.5 mm, 220 parts, among them IC1 OPA4743EA, IC2 OPA2743EA, IC3 OPA2743EA, IC4 OPA4743EA, U1 DRV8302, U10 V_REG_LDOSMD2, U11 MAX881R, U12 V_REG_LDOSMD2, U2 ACS712, U3 ACS712, U4 V_REG_LDOSMD2, U5 V_REG_LDOSMD2, U6 MAX881R, U7 DRV8302, U8 ACS712, U9 ACS712

Commit message: New merged TinyHusk submitted for fab on 3/26
Parts:
- removed C75, C76, C77, C78, C79: 10uF, SparkFun:1210
- removed C80: 10uF, dan-rcl:0603
- removed IC3: OPA2743EA, linear:MSOP08
- removed IC4: OPA4743EA, linear:TSSOP14
- removed R83: 330R, dan-rcl:0603
- removed R84: 6.8K, dan-rcl:0603
- removed R85: 22k, dan-rcl:0603
- removed R86: (no value), dan-rcl:0603
- removed U11: MAX881R, xow:UMAX-10
- removed U12: V_REG_LDOSMD2, SparkFun:SC70
- added SJ3: (no value), SparkFun:SJ_2S-TRACE
- added SJ4: (no value), xow:SJ_X
- C15, C16, C45, C52, C55: value 1uF -> 0.1uF
- C17, C56: value 22uF -> 0.1uF; device dan-rcl:0805 -> dan-rcl:0603
- C41, C42: value 0.1uF -> 1uF
- C43: value 0.1uF -> 2.2uF
- C44: value 1uF -> 0.022uF
- C46: value 2.2uF -> 22uF; device dan-rcl:0603 -> dan-rcl:0805
- C47: value 0.022uF -> 6800pF
- C48: value 0.1uF -> 120pF
- C49: value 22uF -> 1uF; device dan-rcl:0805 -> dan-rcl:0603
- C50: value 6800pF -> 22uF; device dan-rcl:0603 -> dan-rcl:0805
- C51: value 120pF -> 10000pF
- C53: value 22uF -> 10000pF; device dan-rcl:0805 -> dan-rcl:0603
- C54: value 1uF -> 10000pF
- C57: value 10000pF -> 0.1uF
- C58, C61, C62, C63: value 0.1uF -> 10uF; device dan-rcl:0603 -> SparkFun:1210
- C59, C60: value 10000pF -> 10uF; device dan-rcl:0603 -> SparkFun:1210
- C74: device SparkFun:1210 -> dan-rcl:0603
- IC2: value OPA2743EA -> OPA4743EA; device linear:MSOP08 -> linear:TSSOP14
- R26: value 1K -> 330R
- R27: value 330R -> 1K
- R28, R29: value 1K -> 22k
- R48, R49: value 22k -> 1mR; device dan-rcl:0603 -> SparkFun:R2512
- R50, R51: value 1mR -> 0R; device SparkFun:R2512 -> dan-rcl:0603
- R56: value 0R -> 91k
- R57: value 0R -> 12k
- R58: value 91k -> 1mR; device dan-rcl:0603 -> SparkFun:R2512
- R59: value 12k -> 1mR; device dan-rcl:0603 -> SparkFun:R2512
- R60: value 1mR -> 205k; device SparkFun:R2512 -> dan-rcl:0603
- R61: value 1mR -> 16.2k; device SparkFun:R2512 -> dan-rcl:0603
- R62: value 205k -> 59k
- R63: value 16.2k -> 10k
- R64: value 59k -> 22k
- R65: value 10k -> 330R
- R66: value 22k -> 1K
- R69, R71, R72: value 1K -> 6.8K
- R73, R76, R79: value 6.8K -> 330R
- R74, R77, R80: value 330R -> 6.8K
- R81: value 6.8K -> 22k
- R82: value 6.8K -> (none)
- SJ1: device SparkFun:SJ_3 -> xow:SJ_X
- SJ2: device SparkFun:SJ_3 -> SparkFun:SJ_2S-TRACE
- U6: value MAX881R -> DRV8302; device xow:UMAX-10 -> xow:HTSSOP-56
- U7: value DRV8302 -> ACS712; device xow:HTSSOP-56 -> SparkFun:SO08
- U9: value ACS712 -> V_REG_LDOSMD2; device SparkFun:SO08 -> SparkFun:SC70
- moved SJ2 94.0 mm to (5.40, 19.1), turned to 90 degrees
- moved R29 86.2 mm to (90.8, 4.76)
- moved R28 73.0 mm to (76.2, 6.99), flipped to the bottom, turned to 270 degrees
- moved C15 66.3 mm to (70.2, 11.4)
- moved C16 66.3 mm to (70.2, 14.0)
- moved C17 58.2 mm to (70.2, 16.5), turned to 90 degrees
- moved U6 57.0 mm to (64.8, 14.0), turned to 90 degrees
- moved IC2 52.3 mm to (62.2, 35.6), flipped to the bottom, turned to 180 degrees
- moved FB3 52.2 mm to (59.7, 43.8), turned to 90 degrees
- moved R62 49.8 mm to (62.2, 6.03)
- moved L2 49.5 mm to (64.8, 2.54), turned to 180 degrees
- moved C67 49.3 mm to (97.2, 35.9), flipped to the bottom
- moved C46 49.2 mm to (59.1, 2.54), turned to 0 degrees
- moved R74 48.6 mm to (57.1, 40.0), turned to 0 degrees
- moved JP4 47.0 mm to (100.3, 24.1), turned to 270 degrees
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Connections:
- removed net -UB: C16.1, IC1.11, IC2.4, U6.3
- removed net -UB1: C55.1, IC3.4, IC4.11, U11.3
- removed net N$81: IC4.6, IC4.7, R81.1
- removed net N$82: IC4.8, IC4.9, R84.1
- removed net N$83: IC4.13, IC4.14, R75.1
- removed net N$84: IC4.3, R73.1, R74.2
- removed net N$85: IC4.10, R76.1, R77.2
- removed net N$86: IC4.5, R79.1, R80.2
- removed net N$87: IC4.12, R82.1, R83.2
- removed net N$88: R85.2, U7.26
- removed net N$89: C62.1, U9.6
- removed net N$90: C63.1, U8.6
- net !PWM_A1: now also U6.18; no longer U7.18
- net !PWM_B1: now also U6.20; no longer U7.20
- net !PWM_C1: now also U6.22; no longer U7.22
- net +3V1: now also C74.1, SJ3.2, U10.5, U6.24; no longer C80.1, U12.5, U7.24
- net +3V3: now also SJ2.2
- net +5V: no longer IC2.8, U6.10, U6.5
- net +5V1: now also C50.1, IC2.4, U10.1, U10.3, U7.8, U9.5; no longer C53.1, IC3.8, IC4.4, U10.5, U11.10, U11.5, U12.1, U12.3, U9.8
- net AGND: now also IC1.11, R24.2, R26.2; no longer C16.2, C17.2, IC2.3, IC2.5, U6.6, U6.8
- net AGND1: now also C41.2, C49.2, C50.2, C51.1, C52.1, C53.1, C54.1, C57.2, C74.2, IC2.11, R65.2, R67.2, U6.28, U7.5, U9.2; no longer C44.2, C52.2, C53.2, C57.1, C58.1, C59.1, C60.1, C61.2, C62.2, C63.2, C80.2, IC3.3, IC3.5, U11.6, U11.8, U12.2, U7.28, U9.5
- net GND2: now also C42.2, C43.2, C47.1, C48.1, R57.1, R60.1, R63.2, R64.2, R82.1, SJ4.1, U6.12, U6.8, U6.9, U6.PWRPAD; no longer C45.2, C49.2, C50.1, C51.1, R59.1, R62.1, R65.2, R66.2, R86.1, SJ2.1, U7.12, U7.8, U7.9, U7.PWRPAD
- net I_A: now also R25.1; no longer IC2.1
- net I_A1: now also R65.1, R66.1; no longer IC3.1, R67.1
- net I_B: now also R26.1; no longer IC2.7
- net I_B1: now also R67.1, R68.1; no longer IC3.7, R70.1
- net I_B_5V: no longer R26.2
- net I_B_5V1: now also R66.2, U8.7; no longer R68.2, R69.2, U9.7
- net I_C_5V: now also R27.2; no longer R28.2, R29.2
- net I_C_5V1: now also R68.2, U7.7; no longer R71.2, R72.2, U8.7
- net I_P1: now also C55.1, R81.1; no longer C61.1, R85.1
- net M_A1: now also C15.2, R28.1, R78.2, U6.46; no longer C41.2, R44.1, R82.2, U7.46
- net M_B1: now also R58.1, U8.3, U8.4; no longer R60.1, U9.3, U9.4
- net M_C1: now also R59.1, U7.3, U7.4; no longer R61.1, U8.3, U8.4
- net N$21: now also SJ2.1
- net N$27: now also R28.2, R50.2; no longer R44.2, R52.2
- net N$28: now also R44.2, R52.2; no longer R46.2, R54.2
- net N$35: now also D11.1, R45.2, R53.2, S_BL1.1; no longer C17.1, U6.7
- net N$37: now also D12.1, R46.2, R54.2, S_CH1.1; no longer C15.1, U6.1
- net N$38: now also D13.1, R47.2, R55.2, S_CL1.1; no longer C15.2, U6.2
- net N$39: now also C15.1, U6.48; no longer IC2.2, R24.2, R25.1, R26.1
- net N$40: now also C16.1, U6.43; no longer IC2.6, R27.2, R28.1, R29.1
- net N$45: now also C17.1, U6.38; no longer D11.1, R47.2, R55.2, S_BL1.1
- net N$49: now also D9.1, R29.2, R51.2, S_AL1.1; no longer D12.1, R48.2, R56.2, S_CH1.1
- net N$50: now also R50.1, U6.47; no longer D13.1, R49.2, R57.2, S_CL1.1
- net N$51: now also R51.1, U6.45; no longer C41.1, U7.48
- net N$52: now also R52.1, U6.42; no longer C42.1, U7.43
- net N$53: now also R53.1, U6.40; no longer C43.1, U7.38
- net N$54: now also R54.1, U6.37; no longer D9.1, R45.2, R53.2, S_AL1.1
- net N$55: now also R55.1, U6.35; no longer R52.1, U7.47
- net N$56: now also SJ4.2, U6.10; no longer R53.1, U7.45
- net N$57: now also C42.1, R56.2, SJ3.1, SJ4.3, U6.16, U6.23; no longer R54.1, U7.42
- net N$58: now also C41.1, U6.27; no longer R55.1, U7.40
- net N$59: now also C43.1, U6.13; no longer R56.1, U7.37
- net N$60: now also C44.2, U6.14; no longer R57.1, U7.35
- net N$61: now also C44.1, U6.15; no longer SJ2.2, U7.10
- net N$62: now also R56.1, R57.2, U6.11; no longer C45.1, R58.2, SJ2.3, U7.16, U7.23
- net N$63: now also C45.2, D14.C, L2.P$2, U6.50, U6.51; no longer C44.1, U7.27
- net N$64: now also C45.1, U6.52; no longer C46.1, U7.13
- net N$65: now also C48.2, R61.1, U6.2; no longer C47.2, U7.14
- net N$66: now also C47.2, R61.2; no longer C47.1, U7.15
- net N$67: now also R60.2, U6.1; no longer R58.1, R59.2, U7.11
- net N$68: now also R62.1, R63.1, U6.3; no longer C48.2, D14.C, L2.P$2, U7.50, U7.51
- net N$69: now also R64.1, U6.7; no longer C48.1, U7.52
- net N$70: now also IC2.1, IC2.2, R74.1; no longer C51.2, R63.1, U7.2
- net N$71: now also IC2.6, IC2.7, R77.1; no longer C50.2, R63.2
- net N$72: now also IC2.8, IC2.9, R80.1; no longer R62.2, U7.1
- net N$73: now also IC2.13, IC2.14, R71.1; no longer R64.1, R65.1, U7.3
- net N$74: now also IC2.3, R69.1, R70.2; no longer R66.1, U7.7
- net N$75: now also IC2.10, R72.1, R73.2; no longer C56.1, U11.7
- net N$76: now also IC2.5, R75.1, R76.2; no longer C54.1, U11.1
- net N$77: now also IC2.12, R78.1, R79.2; no longer C54.2, U11.2
- net N$78: now also R81.2, U6.26; no longer IC3.2, R67.2, R68.1, R69.1
- net N$79: now also C56.1, U8.6; no longer IC3.6, R70.2, R71.1, R72.1
- net N$80: now also C57.1, U7.6; no longer IC4.1, IC4.2, R78.1
- net PWM_A1: now also U6.17; no longer U7.17
- net PWM_B1: now also U6.19; no longer U7.19
- net PWM_C1: now also U6.21; no longer U7.21
- net R_B1: now also C16.2, R44.1, R58.2, R72.2, U6.41, U8.1, U8.2; no longer C42.2, R46.1, R60.2, R76.2, U7.41, U9.1, U9.2
- net R_C1: now also C17.2, R46.1, R59.2, R75.2, U6.36, U7.1, U7.2; no longer C43.2, R48.1, R61.2, R79.2, U7.36, U8.1, U8.2
- net V+1: now also C58.1, C59.1, C60.1, C61.1, C62.1, C63.1, R69.2, U6.29, U6.53, U6.54; no longer C74.1, C75.1, C76.1, C77.1, C78.1, C79.1, R73.2, U7.29, U7.53, U7.54
- net V-1: now also R48.1, R49.1, R70.1, R73.1, R76.1, R79.1, R82.2, U6.31; no longer R50.1, R51.1, R74.1, R77.1, R80.1, R83.1, R86.2, U7.31
- net VCC1: now also C46.1, R62.2, U9.1, U9.3; no longer C52.1, R64.2, U10.1, U10.3
- net V_A1: now also C51.2, R71.2; no longer C57.2, R75.2
- net V_B1: now also C54.2, R80.2; no longer C60.2, R84.2
- net V_C1: now also C53.2, R77.2; no longer C59.2, R81.2
- net V_LOW1: now also C58.2, C59.2, C60.2, C61.2, C62.2, C63.2, R29.1, R48.2, R49.2, U6.30, U6.34, U6.39, U6.44; no longer C74.2, C75.2, C76.2, C77.2, C78.2, C79.2, R49.1, R50.2, R51.2, U7.30, U7.34, U7.39, U7.44
- net V_P1: now also C52.2, R74.2; no longer C58.2, R78.2
Routing:
- net N$51: track 1.91 -> 37.1 mm, vias 0 -> 1
- net N$60: track 35.6 -> 2.77 mm, vias 1 -> 0
- net N$56: track 36.9 -> 7.10 mm
- net N$88: track 24.7 -> 0.00 mm, vias 2 -> 0
- net -UB1: track 21.9 -> 0.00 mm, vias 2 -> 0
- net -UB: track 21.9 -> 0.00 mm, vias 2 -> 0
- net N$55: track 14.4 -> 36.3 mm, vias 0 -> 1
- net N$53: track 1.88 -> 23.7 mm, vias 0 -> 1
- net N$58: track 24.2 -> 3.72 mm, vias 1 -> 0
- net N$78: track 4.62 -> 23.8 mm, vias 0 -> 2
- net N$59: track 20.7 -> 2.61 mm
- net N$54: track 5.87 -> 20.8 mm
- net +5V1: track 85.8 -> 73.9 mm, vias 2 -> 1
- net +5V: track 85.8 -> 73.9 mm, vias 2 -> 1
- net N$62: track 17.0 -> 5.54 mm
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Other:
- board size 101.6 x 49.5 mm -> 102.9 x 49.5 mm
- board text added: "03/2012"
- board text added: "5"
- board text added: "Husk"
- board text added: "Tiny"
- board text added: "v2.1"
- board text removed: "02/2012"
- board text removed: "Xo Wang"
- board text removed: "v2.0a"
