File: TinyHusk/TinyHusk.brd (EAGLE design)
At the start: 49.5 x 49.5 mm, 110 parts, among them IC1 OPA4743EA, IC2 OPA2743EA, U1 DRV8302, U2 ACS712, U3 ACS712, U4 V_REG_LDOSMD2, U5 V_REG_LDOSMD2, U6 MAX881R

Commit message: Iterated TinyHusk to v2.1
Parts:
- removed C15, C16: 1uF, dan-rcl:0603
- removed C17: 22uF, dan-rcl:0805
- removed IC2: OPA2743EA, linear:MSOP08
- removed R28, R29: 1K, dan-rcl:0603
- removed U6: MAX881R, xow:UMAX-10
- added SJ2: (no value), SparkFun:SJ_2S-TRACE
- R26: value 1K -> 330R
- R27: value 330R -> 1K
- SJ1: device SparkFun:SJ_3 -> xow:SJ_X
- moved R26 9.55 mm to (10.2, 34.9), turned to 0 degrees
- moved SJ1 8.24 mm to (6.99, 16.2), flipped to the top, turned to 0 degrees
- moved R27 2.01 mm to (9.53, 36.8), turned to 90 degrees
- moved C10 1.14 mm to (4.13, 6.99)
- moved C5 1.00 mm to (4.13, 13.7), turned to 90 degrees
- moved R15 1.00 mm to (4.13, 11.4)
- moved R16 1.00 mm to (4.13, 9.21)
- moved R20 0.90 mm to (5.71, 6.99)
- moved C11 0.71 mm to (5.71, 9.21)
- moved C6 0.71 mm to (5.71, 11.4)
- moved C7 0.71 mm to (5.71, 13.7)
- moved R19 0.63 mm to (5.08, 4.45)
- moved C1 0.32 mm to (16.8, 11.4)
- moved C2 0.32 mm to (16.8, 14.0)
- moved C3 0.32 mm to (16.8, 16.5)
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Connections:
- removed net -UB: C16.1, IC1.11, IC2.4, U6.3
- removed net N$35: C17.1, U6.7
- removed net N$37: C15.1, U6.1
- removed net N$38: C15.2, U6.2
- removed net N$39: IC2.2, R24.2, R25.1, R26.1
- removed net N$40: IC2.6, R27.2, R28.1, R29.1
- net +3V3: now also SJ2.2
- net +5V: no longer IC2.8, U6.10, U6.5
- net AGND: now also IC1.11, R24.2, R26.2; no longer C16.2, C17.2, IC2.3, IC2.5, U6.6, U6.8
- net I_A: now also R25.1; no longer IC2.1
- net I_B: now also R26.1; no longer IC2.7
- net I_B_5V: no longer R26.2
- net I_C_5V: now also R27.2; no longer R28.2, R29.2
- net N$21: now also SJ2.1
Routing:
- net -UB: track 21.9 -> 0.00 mm, vias 2 -> 0
- net +5V: track 85.8 -> 73.9 mm, vias 2 -> 1
- net VCC: track 36.7 -> 31.7 mm
- net N$39: track 4.62 -> 0.00 mm
- net N$40: track 4.35 -> 0.00 mm
- net +3V3: track 9.64 -> 12.8 mm
- net N$37: track 2.08 -> 0.00 mm
- net N$35: track 1.92 -> 0.00 mm
- net N$38: track 1.69 -> 0.00 mm
- net I_B_5V: track 4.22 -> 2.95 mm
- net V+: track 63.0 -> 64.3 mm
- net V_LOW: track 29.0 -> 30.3 mm
- net N$3: track 24.7 -> 23.8 mm
- net PWM_A: track 10.7 -> 9.94 mm
- net N$19: track 35.6 -> 36.3 mm
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Other:
- board text added: "03/2012"
- board text added: "5"
- board text added: "Husk"
- board text added: "Tiny"
- board text added: "v2.1"
- board text removed: "02/2012"
- board text removed: "Xo Wang"
- board text removed: "v2.0a"

Commit message: Change values of I_B & I_C resistor dividers
Parts:
- R24, R26: value 330R -> 4.7k
- R25, R27: value 1K -> 9.1k
Changed lines of the file:
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@@
 <layer number="27" name="tValues" color="7" fill="1" visible="no" active="yes"/>
 <layer number="28" name="bValues" color="7" fill="1" visible="no" active="yes"/>
-<layer number="29" name="tStop" color="7" fill="3" visible="yes" active="yes"/>
-<layer number="30" name="bStop" color="7" fill="6" visible="yes" active="yes"/>
+<layer number="29" name="tStop" color="7" fill="3" visible="no" active="yes"/>
+<layer number="30" name="bStop" color="7" fill="6" visible="no" active="yes"/>
 <layer number="31" name="tCream" color="7" fill="4" visible="no" active="yes"/>
 <layer number="32" name="bCream" color="7" fill="5" visible="no" active="yes"/>
@@
 <layer number="144" name="Drill_legend" color="7" fill="1" visible="no" active="yes"/>
 <layer number="151" name="HeatSink" color="7" fill="1" visible="no" active="yes"/>
-<layer number="200" name="200bmp" color="7" fill="10" visible="yes" active="yes"/>
-<layer number="201" name="201bmp" color="7" fill="10" visible="yes" active="yes"/>
+<layer number="200" name="200bmp" color="7" fill="10" visible="no" active="yes"/>
+<layer number="201" name="201bmp" color="7" fill="10" visible="no" active="yes"/>
 <layer number="202" name="202bmp" color="3" fill="10" visible="no" active="yes"/>
 <layer number="203" name="203bmp" color="4" fill="10" visible="no" active="yes"/>
@@
 <element name="C12" library="dan-rcl" package="0603" value="1uF" x="3.81" y="22.86" rot="R270"/>
 <element name="C13" library="dan-rcl" package="0805" value="22uF" x="6.35" y="25.4" rot="R180"/>
-<element name="R24" library="dan-rcl" package="0603" value="330R" x="10.16" y="27.305"/>
-<element name="R25" library="dan-rcl" package="0603" value="1K" x="10.795" y="25.4" rot="R270"/>
-<element name="R26" library="dan-rcl" package="0603" value="330R" x="10.16" y="34.925"/>
-<element name="R27" library="dan-rcl" package="0603" value="1K" x="9.525" y="36.83" rot="R90"/>
+<element name="R24" library="dan-rcl" package="0603" value="4.7k" x="10.16" y="27.305"/>
+<element name="R25" library="dan-rcl" package="0603" value="9.1k" x="10.795" y="25.4" rot="R270"/>
+<element name="R26" library="dan-rcl" package="0603" value="4.7k" x="10.16" y="34.925"/>
+<element name="R27" library="dan-rcl" package="0603" value="9.1k" x="9.525" y="36.83" rot="R90"/>
 <element name="IC1" library="linear" package="TSSOP14" value="OPA4743EA" x="8.89" y="35.56" rot="MR180"/>
 <element name="R30" library="dan-rcl" package="0603" value="6.8K" x="8.255" y="40.64" rot="MR90"/>

Commit message: Iterate to v2.2; just fix silkscreen labels for PWM inputs
Other:
- board text added: "04/2012"
- board text added: "v2.2"
- board text removed: "03/2012"
- board text removed: "v2.1"
Changed lines of the file:
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@@
 <text x="2.54" y="48.26" size="2.54" layer="22" font="vector" ratio="17" rot="MR180">-</text>
 <text x="43.18" y="2.54" size="2.54" layer="22" font="vector" ratio="17" rot="MR180">+</text>
-<text x="7.62" y="44.45" size="1.27" layer="29" font="vector" ratio="17">03/2012</text>
-<text x="24.13" y="0.3175" size="1.778" layer="30" font="vector" ratio="17" rot="MR0">v2.1</text>
+<text x="7.62" y="44.45" size="1.27" layer="29" font="vector" ratio="17">04/2012</text>
+<text x="24.13" y="0.3175" size="1.778" layer="30" font="vector" ratio="17" rot="MR0">v2.2</text>
 <text x="2.2225" y="10.795" size="1.27" layer="22" font="vector" ratio="17" rot="MR180">A</text>
-<text x="2.2225" y="13.335" size="1.27" layer="22" font="vector" ratio="17" rot="MR180">B</text>
-<text x="2.2225" y="15.875" size="1.27" layer="22" font="vector" ratio="17" rot="MR180">C</text>
-<text x="2.2225" y="18.415" size="1.27" layer="22" font="vector" ratio="17" rot="MR180">!A</text>
-<text x="2.2225" y="20.955" size="1.27" layer="22" font="vector" ratio="17" rot="MR180">!B</text>
+<text x="2.2225" y="13.335" size="1.27" layer="22" font="vector" ratio="17" rot="MR180">!A</text>
+<text x="2.2225" y="15.875" size="1.27" layer="22" font="vector" ratio="17" rot="MR180">B</text>
+<text x="2.2225" y="18.415" size="1.27" layer="22" font="vector" ratio="17" rot="MR180">!B</text>
+<text x="2.2225" y="20.955" size="1.27" layer="22" font="vector" ratio="17" rot="MR180">C</text>
 <text x="2.2225" y="23.495" size="1.27" layer="22" font="vector" ratio="17" rot="MR180">!C</text>
 <text x="2.2225" y="26.035" size="1.27" layer="22" font="vector" ratio="17" rot="MR180">IB</text>
