File: TinyHusk/TinyHusk.sch (EAGLE design)
At the start: 110 parts, among them IC1 OPA4743EA, IC2 OPA2743EA, U1 DRV8302, U2 ACS712, U3 ACS712, U4 V_REG_LDOSMD2, U5 V_REG_LDOSMD2, U6 MAX881R

Commit message: Iterated TinyHusk to v2.1
Parts:
- removed C15, C16: 1uF, dan-rcl:C0603
- removed C17: 22uF, dan-rcl:C0805
- removed IC2: OPA2743EA, linear:OPA2743EA
- removed R28, R29: 1K, dan-rcl:R0603
- removed U6: MAX881R, xow:MAX881R
- added SJ2: SOLDERJUMPERTRACE, SparkFun:SOLDERJUMPERTRACE
- R26: value 1K -> 330R
- R27: value 330R -> 1K
- SJ1: device SparkFun:SOLDERJUMPER_2WAYS -> xow:SOLDERJUMPER_2WAYS
Connections:
- removed net -UB: C16.1, IC1P.V-, IC2P.V-, U6.NEGOUT
- removed net N$35: C17.1, U6.OUT
- removed net N$37: C15.1, U6.C1+
- removed net N$38: C15.2, U6.C1-
- removed net N$39: IC2A.-IN, R24.2, R25.1, R26.1
- removed net N$40: IC2B.-IN, R27.2, R28.1, R29.1
- net +3V3: now also SJ2.2
- net +5V: no longer IC2P.V+, U6.!SHDN, U6.IN
- net AGND: now also IC1P.V-, R24.2, R26.2; no longer C16.2, C17.2, IC2A.+IN, IC2B.+IN, U6.FB, U6.GND
- net I_A: now also R25.1; no longer IC2A.OUT
- net I_B: now also R26.1; no longer IC2B.OUT
- net I_B_5V: no longer R26.2
- net I_C_5V: now also R27.2; no longer R28.2, R29.2
- net N$21: now also SJ2.1
Other:
- moved on the sheet: R24, R25, R26, R27

Commit message: Change values of I_B & I_C resistor dividers
Parts:
- R24, R26: value 330R -> 4.7k
- R25, R27: value 1K -> 9.1k
Changed lines of the file:
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@@
 <part name="C12" library="dan-rcl" deviceset="C" device="0603" value="1uF"/>
 <part name="C13" library="dan-rcl" deviceset="C" device="0805" value="22uF"/>
-<part name="R24" library="dan-rcl" deviceset="R" device="0603" value="330R"/>
-<part name="R25" library="dan-rcl" deviceset="R" device="0603" value="1K"/>
-<part name="R26" library="dan-rcl" deviceset="R" device="0603" value="330R"/>
-<part name="R27" library="dan-rcl" deviceset="R" device="0603" value="1K"/>
+<part name="R24" library="dan-rcl" deviceset="R" device="0603" value="4.7k"/>
+<part name="R25" library="dan-rcl" deviceset="R" device="0603" value="9.1k"/>
+<part name="R26" library="dan-rcl" deviceset="R" device="0603" value="4.7k"/>
+<part name="R27" library="dan-rcl" deviceset="R" device="0603" value="9.1k"/>
 <part name="AGND9" library="supply1" deviceset="AGND" device=""/>
 <part name="IC1" library="linear" deviceset="OPA4743" device="EA"/>

Commit message: Iterate to v2.2; just fix silkscreen labels for PWM inputs
Parts:
- S_AH, S_AL, S_BH, S_BL, S_CH, S_CL: device xow:MOSFET-N_D2PAK-7 -> xow:MOSFET-ND2PAK7
Changed lines of the file:
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@@
 <part name="U1" library="xow" deviceset="DRV8302" device=""/>
 <part name="GND1" library="supply1" deviceset="GND" device=""/>
-<part name="S_AH" library="xow" deviceset="MOSFET-N_D2PAK-7" device="" value="D2PAK-7"/>
-<part name="S_AL" library="xow" deviceset="MOSFET-N_D2PAK-7" device="" value="D2PAK-7"/>
-<part name="S_BH" library="xow" deviceset="MOSFET-N_D2PAK-7" device="" value="D2PAK-7"/>
-<part name="S_BL" library="xow" deviceset="MOSFET-N_D2PAK-7" device="" value="D2PAK-7"/>
-<part name="S_CH" library="xow" deviceset="MOSFET-N_D2PAK-7" device="" value="D2PAK-7"/>
-<part name="S_CL" library="xow" deviceset="MOSFET-N_D2PAK-7" device="" value="D2PAK-7"/>
+<part name="S_AH" library="xow" deviceset="MOSFET-N" device="D2PAK7" value="D2PAK-7"/>
+<part name="S_AL" library="xow" deviceset="MOSFET-N" device="D2PAK7" value="D2PAK-7"/>
+<part name="S_BH" library="xow" deviceset="MOSFET-N" device="D2PAK7" value="D2PAK-7"/>
+<part name="S_BL" library="xow" deviceset="MOSFET-N" device="D2PAK7" value="D2PAK-7"/>
+<part name="S_CH" library="xow" deviceset="MOSFET-N" device="D2PAK7" value="D2PAK-7"/>
+<part name="S_CL" library="xow" deviceset="MOSFET-N" device="D2PAK7" value="D2PAK-7"/>
 <part name="C1" library="dan-rcl" deviceset="C" device="0603" value="0.1uF"/>
 <part name="C2" library="dan-rcl" deviceset="C" device="0603" value="0.1uF"/>
